File: z280-s100.kicad_pcb (KiCad board)
At the start: 2 copper layers, 254 x 134.6 mm, 33 parts, among them J1 S-100 edge, J2 JTAG (1x6), J3 JP VPP, J4 JP A15, J5 JP A16, J6 JP A17/VDD, J7 JP PGM, J8 JP VDD, U1 Z280 (PLCC-68), U10 SRAM bank0 odd, U11 27SF020 even, U12 27SF020 odd, U13 MAX232, U14 DS1813 reset, U15 7805, U16 74HCT245 addr0, U17 74HCT245 addr1, U18 74HCT245 addr2, U19 74HCT245 status, U2 ATF1508 control, U20 74HCT245 control, U21 74HCT245 pHLDA, U22 SRAM bank1 even, U23 SRAM bank1 odd, U24 ATF1508 data, U3 74HC573 lo, U4 74HC573 hi, U9 SRAM bank0 even, Y1 24 MHz crystal

Commit message: Z280 S-100: 4-layer PCB with power planes and edge-connector test points
gen_pcb.py now emits a 4-layer board (In1.Cu = GND plane, In2.Cu = +5V
plane), imports the S-100 edge connector geometry from the Z80 V3
reference board, and adds a row of test-point vias above each connector
finger. Component reference designators are synced to the schematic's
current annotation (the edge connector is J8). The schematic generator
gained the serial header and symbol text/body layout fixes, and the
schematic, netlist, and PCB were regenerated.

Co-Authored-By: Claude <noreply@anthropic.com>
Parts:
- removed U21: 74HCT245 pHLDA, DIP-20
- removed U22: SRAM bank1 even, DIP-32
- removed U23: SRAM bank1 odd, DIP-32
- removed U24: ATF1508 data, Package_LCC:PLCC-84_THT-Socket
- added J9: JTAG (1x6), HDR-6, F.Cu at (25.0, 30.0)
- added U5: ATF1508 data, Package_LCC:PLCC-84_THT-Socket, F.Cu at (225.0, 85.0)
- added U6: SRAM bank0 even, DIP-32, F.Cu at (60.0, 52.0)
- added U7: SRAM bank0 odd, DIP-32, F.Cu at (60.0, 34.0)
- added U8: SRAM bank1 even, DIP-32, F.Cu at (140.0, 52.0)
- J1: value S-100 edge -> JP VPP; footprint S100_MALE -> HDR-2
- J2: value JTAG (1x6) -> JP A15; footprint HDR-6 -> HDR-2
- J3: value JP VPP -> JP A16
- J4: value JP A15 -> JP A17/VDD
- J5: value JP A16 -> JP PGM
- J6: value JP A17/VDD -> JP VDD
- J7: value JP PGM -> Serial (2x5); footprint HDR-2 -> Connector_PinHeader_2.54mm:PinHeader_2x05_P2.54mm_Vertical
- J8: value JP VDD -> S-100 edge; footprint HDR-2 -> S100_MALE
- U10: value SRAM bank0 odd -> 27SF020 even
- U11: value 27SF020 even -> 27SF020 odd
- U12: value 27SF020 odd -> 7805; footprint DIP-32 -> HDR-3
- U13: value MAX232 -> DS1813 reset; footprint DIP-16 -> HDR-3
- U14: value DS1813 reset -> MAX232; footprint HDR-3 -> DIP-16
- U15: value 7805 -> 74HCT245 addr0; footprint HDR-3 -> DIP-20
- U16: value 74HCT245 addr0 -> 74HCT245 addr1
- U17: value 74HCT245 addr1 -> 74HCT245 addr2
- U18: value 74HCT245 addr2 -> 74HCT245 status
- U19: value 74HCT245 status -> 74HCT245 control
- U2: value ATF1508 control -> 74HC573 lo; footprint Package_LCC:PLCC-84_THT-Socket -> DIP-20
- U20: value 74HCT245 control -> 74HCT245 pHLDA
- U3: value 74HC573 lo -> 74HC573 hi
- U4: value 74HC573 hi -> ATF1508 control; footprint DIP-20 -> Package_LCC:PLCC-84_THT-Socket
- U9: value SRAM bank0 even -> SRAM bank1 odd
- moved U13 233.9 mm to (252.0, 120.0)
- moved U14 233.9 mm to (20.0, 90.0)
- moved J7 200.0 mm to (20.0, 70.0)
- moved J8 195.8 mm to (50.8, 157.5)
- moved J2 184.0 mm to (205.0, 68.0)
- moved J1 174.0 mm to (200.0, 68.0)
- moved U10 166.0 mm to (225.0, 52.0)
- moved U15 162.0 mm to (90.0, 133.0)
- moved U2 106.4 mm to (45.0, 133.0)
- moved U12 104.5 mm to (252.0, 135.0), turned to 0 degrees
- moved U4 89.0 mm to (140.0, 85.0)
- moved U9 82.0 mm to (140.0, 34.0)
- moved U16 20.0 mm to (110.0, 133.0)
- moved U17 20.0 mm to (130.0, 133.0)
- moved U18 20.0 mm to (150.0, 133.0)
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Connections:
- J1 pad 1: +8V -> FLASH_VPP
- J1 pad 2: +16V -> +5V
- J2 pad 1: JTAG_TCK -> FLASH_A15
- J2 pad 2: JTAG_TMS -> A16
- J3 pad 1: FLASH_VPP -> FLASH_A16
- J3 pad 2: +5V -> A17
- J4 pad 1: FLASH_A15 -> FLASH_A17
- J4 pad 2: A16 -> A18
- J5 pad 1: FLASH_A16 -> FLASH_PGM
- J5 pad 2: A17 -> +5V
- J6 pad 1: FLASH_A17 -> FLASH_VDD
- J6 pad 2: A18 -> +5V
- J7 pad 1: FLASH_PGM -> MAX_RS232_TX
- J7 pad 2: +5V -> MAX_RS232_RX
- J8 pad 1: FLASH_VDD -> +8V
- J8 pad 2: +5V -> +16V
- U1 pad 11: (no net) -> unconnected-(U1-DMASTB0-Pad11)
- U1 pad 13: (no net) -> unconnected-(U1-DMASTB1-Pad13)
- U1 pad 20: (no net) -> unconnected-(U1-CTIO1-Pad20)
- U1 pad 23: (no net) -> unconnected-(U1-CTIO2-Pad23)
- U1 pad 25: (no net) -> unconnected-(U1-CTIN2-Pad25)
- U1 pad 26: (no net) -> unconnected-(U1-INT-C-Pad26)
- U1 pad 30: (no net) -> unconnected-(U1-CTIO0/GREQ-Pad30)
- U1 pad 32: (no net) -> unconnected-(U1-CTIN0/GACK-Pad32)
- U1 pad 33: (no net) -> unconnected-(U1-PAUSE-Pad33)
- U1 pad 36: (no net) -> unconnected-(U1-INT-B/EOP-B-Pad36)
- U1 pad 41: (no net) -> unconnected-(U1-CTIN1-Pad41)
- U1 pad 52: (no net) -> unconnected-(U1-RESERVED-Pad52)
- U1 pad 55: (no net) -> unconnected-(U1-RDY0-Pad55)
- U1 pad 56: (no net) -> unconnected-(U1-RDY1-Pad56)
- U1 pad 58: (no net) -> unconnected-(U1-RDY3-Pad58)
- U1 pad 63: (no net) -> unconnected-(U1-RDY2-Pad63)
- U10 pad 1: LA15 -> FLASH_VPP
- U10 pad 10: SRAM_A0 -> LA3
- U10 pad 11: AD0 -> LA2
- U10 pad 12: AD1 -> LA1
- U10 pad 13: AD2 -> AD8
- U10 pad 14: GND -> AD9
- U10 pad 15: AD3 -> AD10
- U10 pad 16: AD4 -> GND
- U10 pad 17: AD5 -> AD11
- U10 pad 18: AD6 -> AD12
- U10 pad 19: AD7 -> AD13
- U10 pad 2: LA13 -> FLASH_A16
- U10 pad 20: MEM_CE0 -> AD14
- U10 pad 21: LA11 -> AD15
- U10 pad 22: MEM_OE -> FLASH_CE
- U10 pad 23: LA12 -> LA11
- U10 pad 24: LA10 -> FLASH_OE
- U10 pad 25: LA9 -> LA12
- U10 pad 26: LA14 -> LA10
- U10 pad 27: MEM_WE_H -> LA9
- U10 pad 28: +5V -> LA14
- U10 pad 29: A19 -> LA15
- U10 pad 3: LA8 -> FLASH_A15
- U10 pad 30: A18 -> FLASH_A17
- U10 pad 31: A17 -> FLASH_PGM
- U10 pad 32: A16 -> FLASH_VDD
- U10 pad 4: LA7 -> LA13
- U10 pad 5: LA6 -> LA8
- U10 pad 6: LA5 -> LA7
- U10 pad 7: LA4 -> LA6
- U10 pad 8: LA3 -> LA5
- U10 pad 9: SRAM_A1 -> LA4
- U11 pad 13: AD8 -> AD0
- U11 pad 14: AD9 -> AD1
- U11 pad 15: AD10 -> AD2
- U11 pad 17: AD11 -> AD3
- U11 pad 18: AD12 -> AD4
- U11 pad 19: AD13 -> AD5
- U11 pad 20: AD14 -> AD6
- U11 pad 21: AD15 -> AD7
- U12 pad 1: FLASH_VPP -> +8V
- U12 pad 2: FLASH_A16 -> GND
- U12 pad 3: FLASH_A15 -> +5V
- U13 pad 1: MAX_C1P -> GND
- U13 pad 2: MAX_VP -> Z_RESET
- U13 pad 3: MAX_C1M -> +5V
- U14 pad 1: GND -> MAX_C1P
- U14 pad 2: Z_RESET -> MAX_VP
- U14 pad 3: +5V -> MAX_C1M
- U15 pad 1: +8V -> S100_A_DIR
- U15 pad 2: GND -> BYTE_SEL
- U15 pad 3: +5V -> LA1
- U16 pad 11: S100_A0 -> S100_A8
- U16 pad 12: S100_A1 -> S100_A9
- U16 pad 13: S100_A2 -> S100_A10
- U16 pad 14: S100_A3 -> S100_A11
- U16 pad 15: S100_A4 -> S100_A12
- U16 pad 16: S100_A5 -> S100_A13
- U16 pad 17: S100_A6 -> S100_A14
- U16 pad 18: S100_A7 -> S100_A15
- U16 pad 2: BYTE_SEL -> LA8
- U16 pad 3: LA1 -> LA9
- U16 pad 4: LA2 -> LA10
- U16 pad 5: LA3 -> LA11
- U16 pad 6: LA4 -> LA12
- U16 pad 7: LA5 -> LA13
- U16 pad 8: LA6 -> LA14
- U16 pad 9: LA7 -> LA15
- U17 pad 11: S100_A8 -> S100_A16
- U17 pad 12: S100_A9 -> S100_A17
- U17 pad 13: S100_A10 -> S100_A18
- U17 pad 14: S100_A11 -> S100_A19
- U17 pad 15: S100_A12 -> S100_A20
- U17 pad 16: S100_A13 -> S100_A21
- U17 pad 17: S100_A14 -> S100_A22
- U17 pad 18: S100_A15 -> S100_A23
- U17 pad 2: LA8 -> A16
- U17 pad 3: LA9 -> A17
- U17 pad 4: LA10 -> A18
- U17 pad 5: LA11 -> A19
- U17 pad 6: LA12 -> A20
- U17 pad 7: LA13 -> A21
- U17 pad 8: LA14 -> A22
- U17 pad 9: LA15 -> A23
- U18 pad 1: S100_A_DIR -> S100_SC_DIR
- U18 pad 11: S100_A16 -> S100_sMEMR
- U18 pad 12: S100_A17 -> S100_sWO
- U18 pad 13: S100_A18 -> S100_sINP
- U18 pad 14: S100_A19 -> S100_sOUT
- U18 pad 15: S100_A20 -> S100_sINTA
- U18 pad 16: S100_A21 -> S100_sHLTA
- U18 pad 17: S100_A22 -> S100_sXTRQ
- U18 pad 18: S100_A23 -> unconnected-(U18-B7-Pad18)
- U18 pad 19: S100_A_OE -> S100_S_OE
- U18 pad 2: A16 -> CPLD_sMEMR
- U18 pad 3: A17 -> CPLD_sWO
- U18 pad 4: A18 -> CPLD_sINP
- U18 pad 5: A19 -> CPLD_sOUT
- U18 pad 6: A20 -> CPLD_sINTA
- U18 pad 7: A21 -> CPLD_sHLTA
- U18 pad 8: A22 -> CPLD_sXTRQ
- U18 pad 9: A23 -> unconnected-(U18-A7-Pad9)
- U19 pad 11: S100_sMEMR -> S100_pSYNC
- U19 pad 12: S100_sWO -> S100_pSTVAL
- U19 pad 13: S100_sINP -> S100_pDBIN
- U19 pad 14: S100_sOUT -> S100_pWR
- U19 pad 15: S100_sINTA -> unconnected-(U19-B4-Pad15)
- U19 pad 16: S100_sHLTA -> unconnected-(U19-B5-Pad16)
- U19 pad 17: S100_sXTRQ -> unconnected-(U19-B6-Pad17)
- U19 pad 18: (no net) -> unconnected-(U19-B7-Pad18)
- U19 pad 19: S100_S_OE -> S100_C_OE
- U19 pad 2: CPLD_sMEMR -> CPLD_pSYNC
- U19 pad 3: CPLD_sWO -> CPLD_pSTVAL
- U19 pad 4: CPLD_sINP -> CPLD_pDBIN
- U19 pad 5: CPLD_sOUT -> CPLD_pWR
- U19 pad 6: CPLD_sINTA -> unconnected-(U19-A4-Pad6)
- U19 pad 7: CPLD_sHLTA -> unconnected-(U19-A5-Pad7)
- U19 pad 8: CPLD_sXTRQ -> unconnected-(U19-A6-Pad8)
- U19 pad 9: (no net) -> unconnected-(U19-A7-Pad9)
- U2 pad 1: Z_AS -> GND
- U2 pad 10: Z_ST3 -> GND
- U2 pad 11: Z_IE -> LATCH_LE
- U2 pad 12: Z_OE -> LA0
- U2 pad 13: +5V -> LA1
- U2 pad 14: JTAG_TDI -> LA2
- U2 pad 15: Z_BUSACK -> LA3
- U2 pad 16: Z_RESET -> LA4
- U2 pad 17: S100_INT -> LA5
- U2 pad 18: S100_NMI -> LA6
- U2 pad 19: GND -> LA7
- U2 pad 2: Z_DS -> AD0
- U2 pad 20: S100_HOLD -> +5V
- U2 pad 3: +5V -> AD1
- U2 pad 4: Z_RW -> AD2
- U2 pad 5: Z_BW -> AD3
- U2 pad 6: Z_ST0 -> AD4
- U2 pad 7: GND -> AD5
- U2 pad 8: Z_ST1 -> AD6
- U2 pad 9: Z_ST2 -> AD7
- U20 pad 1: S100_SC_DIR -> +5V
- U20 pad 11: S100_pSYNC -> S100_pHLDA
- U20 pad 12: S100_pSTVAL -> unconnected-(U20-B1-Pad12)
- U20 pad 13: S100_pDBIN -> unconnected-(U20-B2-Pad13)
- U20 pad 14: S100_pWR -> unconnected-(U20-B3-Pad14)
- U20 pad 15: (no net) -> unconnected-(U20-B4-Pad15)
- U20 pad 16: (no net) -> unconnected-(U20-B5-Pad16)
- U20 pad 17: (no net) -> unconnected-(U20-B6-Pad17)
- U20 pad 18: (no net) -> unconnected-(U20-B7-Pad18)
- U20 pad 19: S100_C_OE -> GND
- U20 pad 2: CPLD_pSYNC -> CPLD_pHLDA
- U20 pad 3: CPLD_pSTVAL -> GND
- U20 pad 4: CPLD_pDBIN -> GND
- U20 pad 5: CPLD_pWR -> GND
- U20 pad 6: (no net) -> GND
- U20 pad 7: (no net) -> GND
- U20 pad 8: (no net) -> GND
- U20 pad 9: (no net) -> GND
- U3 pad 12: LA0 -> LA8
- U3 pad 13: LA1 -> LA9
- U3 pad 14: LA2 -> LA10
- U3 pad 15: LA3 -> LA11
- U3 pad 16: LA4 -> LA12
- U3 pad 17: LA5 -> LA13
- U3 pad 18: LA6 -> LA14
- U3 pad 19: LA7 -> LA15
- U3 pad 2: AD0 -> AD8
- U3 pad 3: AD1 -> AD9
- U3 pad 4: AD2 -> AD10
- U3 pad 5: AD3 -> AD11
- U3 pad 6: AD4 -> AD12
- U3 pad 7: AD5 -> AD13
- U3 pad 8: AD6 -> AD14
- U3 pad 9: AD7 -> AD15
- U4 pad 1: GND -> Z_AS
- U4 pad 10: GND -> Z_ST3
- U4 pad 11: LATCH_LE -> Z_IE
- U4 pad 12: LA8 -> Z_OE
- U4 pad 13: LA9 -> +5V
- U4 pad 14: LA10 -> JTAG_TDI
- U4 pad 15: LA11 -> Z_BUSACK
- U4 pad 16: LA12 -> Z_RESET
- U4 pad 17: LA13 -> S100_INT
- U4 pad 18: LA14 -> S100_NMI
- U4 pad 19: LA15 -> GND
- U4 pad 2: AD8 -> Z_DS
- U4 pad 20: +5V -> S100_HOLD
- U4 pad 3: AD9 -> +5V
- U4 pad 4: AD10 -> Z_RW
- U4 pad 5: AD11 -> Z_BW
- U4 pad 6: AD12 -> Z_ST0
- U4 pad 7: AD13 -> GND
- U4 pad 8: AD14 -> Z_ST1
- U4 pad 9: AD15 -> Z_ST2
- U9 pad 11: AD8 -> AD0
- U9 pad 12: AD9 -> AD1
- U9 pad 13: AD10 -> AD2
- U9 pad 15: AD11 -> AD3
- U9 pad 16: AD12 -> AD4
- U9 pad 17: AD13 -> AD5
- U9 pad 18: AD14 -> AD6
- U9 pad 19: AD15 -> AD7
- U9 pad 20: MEM_CE0 -> MEM_CE1
- U9 pad 27: MEM_WE_L -> MEM_WE_H
Routing:
- net unconnected-(J8-NC-Pad71): vias 0 -> 1
- net unconnected-(J8-NC-Pad69): vias 0 -> 1
- net unconnected-(J8-NC-Pad66): vias 0 -> 1
- net unconnected-(J8-NC-Pad65): vias 0 -> 1
- net unconnected-(J8-NC-Pad28): vias 0 -> 1
- net unconnected-(J8-NC-Pad27): vias 0 -> 1
- net unconnected-(J8-NC-Pad21): vias 0 -> 1
- net S100_sXTRQ: vias 0 -> 1
- net S100_sWO: vias 0 -> 1
- net S100_sOUT: vias 0 -> 1
- net S100_sMEMR: vias 0 -> 1
- net S100_sM1: vias 0 -> 1
- net S100_sINTA: vias 0 -> 1
- net S100_sINP: vias 0 -> 1
- net S100_sHLTA: vias 0 -> 1
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- added copper zone on In2.Cu, net +5V
- added copper zone on In1.Cu, net GND
Other:
- copper layers 2 -> 4

Commit message: Z280 S-100: re-partition CPLDs, external decode, reset/BTI config
Split the two ATF1508s by function: z280-s100-ad.pld (data path) owns
AD0-15 demux/burst/byte-mux, z280-s100-ctl.pld (decider) owns the FSM,
arbitration, memory control and steering. Replace the old
control.pld/data.pld pair.

Move A16-23 decode off-chip to a 74F138 + two 74F521s (SRAM/FLASH/slave
window); drop the 74HC573 latches. Boot ROM is now 2x AT28C256 (word-wide
fetch needs two parts).

Add reset/BTI loading: a 74HCT244 tri-state driver (CFG_OE-gated) drives
AD0-7 during reset, config jumpers J10-J17 strap the BTI value, and a
15-clock hold counter keeps WAIT asserted past reset. Fix dedicated pins
(GCLR/OE1/OE2 tied inactive) and make SIXTN bidirectional.

PCB: RAM/ROM clustered left, decode + BTI + config straps top-right,
data CPLD aligned above the memory column.

Co-Authored-By: Claude <noreply@anthropic.com>
Parts:
- removed J1: JP VPP, HDR-2
- removed J2: JP A15, HDR-2
- removed J3: JP A16, HDR-2
- removed J4: JP A17/VDD, HDR-2
- removed J5: JP PGM, HDR-2
- removed J6: JP VDD, HDR-2
- removed U2: 74HC573 lo, DIP-20
- removed U3: 74HC573 hi, DIP-20
- added C1: 0.1uF, CAP-2, F.Cu at (30.0, 76.0)
- added C10: 0.1uF, CAP-2, F.Cu at (153.0, 122.0)
- added C11: 0.1uF, CAP-2, F.Cu at (172.0, 113.0)
- added C12: 0.1uF, CAP-2, F.Cu at (200.0, 113.0)
- added C13: 0.1uF, CAP-2, F.Cu at (226.0, 113.0)
- added C14: 0.1uF, CAP-2, F.Cu at (85.0, 60.0)
- added C15: 0.1uF, CAP-2, F.Cu at (85.0, 34.0)
- added C16: 0.1uF, CAP-2, F.Cu at (165.0, 60.0)
- added C17: 0.1uF, CAP-2, F.Cu at (165.0, 34.0)
- added C18: 0.1uF, CAP-2, F.Cu at (248.0, 56.0)
- added C19: 0.1uF, CAP-2, F.Cu at (248.0, 34.0)
- added C2: 0.1uF, CAP-2, F.Cu at (30.0, 82.0)
- added C3: 0.1uF, CAP-2, F.Cu at (30.0, 88.0)
- added C4: 0.1uF, CAP-2, F.Cu at (30.0, 94.0)
- added C5: 0.1uF, CAP-2, F.Cu at (30.0, 100.0)
- added C6: 0.1uF, CAP-2, F.Cu at (45.0, 122.0)
- added C7: 0.1uF, CAP-2, F.Cu at (72.0, 122.0)
- added C8: 0.1uF, CAP-2, F.Cu at (99.0, 122.0)
- added C9: 0.1uF, CAP-2, F.Cu at (126.0, 122.0)
- added J10: BTI AD0, HDR-3, F.Cu at (185.0, 108.0)
- added J11: BTI AD1, HDR-3, F.Cu at (195.0, 108.0)
- added J12: BTI AD2, HDR-3, F.Cu at (205.0, 108.0)
- added J13: BTI AD3, HDR-3, F.Cu at (215.0, 108.0)
- added J14: BTI AD4, HDR-3, F.Cu at (225.0, 108.0)
- added J15: BTI AD5, HDR-3, F.Cu at (235.0, 108.0)
- added J16: BTI AD6, HDR-3, F.Cu at (245.0, 108.0)
- added J17: BTI AD7, HDR-3, F.Cu at (255.0, 108.0)
- added U21: 74HCT244 BTI, DIP-20, F.Cu at (172.0, 120.0)
- added U22: 74F138 decode, DIP-16, F.Cu at (200.0, 120.0)
- added U23: 74F521 flash win, DIP-20, F.Cu at (226.0, 120.0)
- added U24: 74F521 slave win, DIP-20, F.Cu at (252.0, 120.0)
- U10: value 27SF020 even -> 28C256 even; footprint DIP-32 -> DIP-28
- U11: value 27SF020 odd -> 28C256 odd; footprint DIP-32 -> DIP-28
- moved U10 90.0 mm to (135.0, 55.0)
- moved U11 90.0 mm to (135.0, 35.0)
- moved U15 55.0 mm to (35.0, 133.0), turned to 90 degrees
- moved U8 50.1 mm to (90.0, 55.0)
- moved U9 50.0 mm to (90.0, 35.0)
- moved U16 48.0 mm to (62.0, 133.0), turned to 90 degrees
- moved U12 45.0 mm to (252.0, 90.0)
- moved U17 41.0 mm to (89.0, 133.0), turned to 90 degrees
- moved U13 40.0 mm to (252.0, 80.0)
- moved Y1 35.0 mm to (252.0, 70.0)
- moved U18 34.0 mm to (116.0, 133.0), turned to 90 degrees
- moved J7 30.3 mm to (16.0, 40.0)
- moved R1 30.0 mm to (252.0, 60.0)
- moved R2 30.0 mm to (252.0, 50.0)
- moved R3 30.0 mm to (252.0, 40.0)
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Connections:
- J8 pad 21: unconnected-(J8-NC-Pad21) -> (no net)
- J8 pad 27: unconnected-(J8-NC-Pad27) -> (no net)
- J8 pad 28: unconnected-(J8-NC-Pad28) -> (no net)
- J8 pad 65: unconnected-(J8-NC-Pad65) -> (no net)
- J8 pad 66: unconnected-(J8-NC-Pad66) -> (no net)
- J8 pad 69: unconnected-(J8-NC-Pad69) -> (no net)
- J8 pad 71: unconnected-(J8-NC-Pad71) -> (no net)
- U1 pad 11: unconnected-(U1-DMASTB0-Pad11) -> (no net)
- U1 pad 13: unconnected-(U1-DMASTB1-Pad13) -> (no net)
- U1 pad 20: unconnected-(U1-CTIO1-Pad20) -> (no net)
- U1 pad 23: unconnected-(U1-CTIO2-Pad23) -> (no net)
- U1 pad 25: unconnected-(U1-CTIN2-Pad25) -> (no net)
- U1 pad 26: unconnected-(U1-INT-C-Pad26) -> (no net)
- U1 pad 30: unconnected-(U1-CTIO0/GREQ-Pad30) -> (no net)
- U1 pad 32: unconnected-(U1-CTIN0/GACK-Pad32) -> (no net)
- U1 pad 33: unconnected-(U1-PAUSE-Pad33) -> (no net)
- U1 pad 36: unconnected-(U1-INT-B/EOP-B-Pad36) -> (no net)
- U1 pad 41: unconnected-(U1-CTIN1-Pad41) -> (no net)
- U1 pad 52: unconnected-(U1-RESERVED-Pad52) -> (no net)
- U1 pad 55: unconnected-(U1-RDY0-Pad55) -> (no net)
- U1 pad 56: unconnected-(U1-RDY1-Pad56) -> (no net)
- U1 pad 58: unconnected-(U1-RDY3-Pad58) -> (no net)
- U1 pad 63: unconnected-(U1-RDY2-Pad63) -> (no net)
- U10 pad 1: FLASH_VPP -> A15
- U10 pad 10: LA3 -> A1
- U10 pad 11: LA2 -> AD8
- U10 pad 12: LA1 -> AD9
- U10 pad 13: AD8 -> AD10
- U10 pad 14: AD9 -> GND
- U10 pad 15: AD10 -> AD11
- U10 pad 16: GND -> AD12
- U10 pad 17: AD11 -> AD13
- U10 pad 18: AD12 -> AD14
- U10 pad 19: AD13 -> AD15
- U10 pad 2: FLASH_A16 -> A13
- U10 pad 20: AD14 -> FLASH_CE
- U10 pad 21: AD15 -> A11
- U10 pad 22: FLASH_CE -> FLASH_OE
- U10 pad 23: LA11 -> A12
- U10 pad 24: FLASH_OE -> A10
- U10 pad 25: LA12 -> A9
- U10 pad 26: LA10 -> A14
- U10 pad 27: LA9 -> FLASH_WE
- U10 pad 28: LA14 -> +5V
- U10 pad 3: FLASH_A15 -> A8
- U10 pad 4: LA13 -> A7
- U10 pad 5: LA8 -> A6
- U10 pad 6: LA7 -> A5
- U10 pad 7: LA6 -> A4
- U10 pad 8: LA5 -> A3
- U10 pad 9: LA4 -> A2
- U11 pad 1: FLASH_VPP -> A15
- U11 pad 10: LA3 -> A1
- U11 pad 11: LA2 -> AD0
- U11 pad 12: LA1 -> AD1
- U11 pad 13: AD0 -> AD2
- U11 pad 14: AD1 -> GND
- U11 pad 15: AD2 -> AD3
- U11 pad 16: GND -> AD4
- U11 pad 17: AD3 -> AD5
- U11 pad 18: AD4 -> AD6
- U11 pad 19: AD5 -> AD7
- U11 pad 2: FLASH_A16 -> A13
- U11 pad 20: AD6 -> FLASH_CE
- U11 pad 21: AD7 -> A11
- U11 pad 22: FLASH_CE -> FLASH_OE
- U11 pad 23: LA11 -> A12
- U11 pad 24: FLASH_OE -> A10
- U11 pad 25: LA12 -> A9
- U11 pad 26: LA10 -> A14
- U11 pad 27: LA9 -> FLASH_WE
- U11 pad 28: LA14 -> +5V
- U11 pad 3: FLASH_A15 -> A8
- U11 pad 4: LA13 -> A7
- U11 pad 5: LA8 -> A6
- U11 pad 6: LA7 -> A5
- U11 pad 7: LA6 -> A4
- U11 pad 8: LA5 -> A3
- U11 pad 9: LA4 -> A2
- U15 pad 1: S100_A_DIR -> S100_DIR
- U15 pad 2: BYTE_SEL -> A0
- U16 pad 1: S100_A_DIR -> S100_DIR
- U17 pad 1: S100_A_DIR -> S100_DIR
- U18 pad 1: S100_SC_DIR -> S100_DIR
- U18 pad 18: unconnected-(U18-B7-Pad18) -> (no net)
- U18 pad 9: unconnected-(U18-A7-Pad9) -> (no net)
- U19 pad 1: S100_SC_DIR -> S100_DIR
- U19 pad 15: unconnected-(U19-B4-Pad15) -> (no net)
- U19 pad 16: unconnected-(U19-B5-Pad16) -> (no net)
- U19 pad 17: unconnected-(U19-B6-Pad17) -> (no net)
- U19 pad 18: unconnected-(U19-B7-Pad18) -> (no net)
- U19 pad 6: unconnected-(U19-A4-Pad6) -> (no net)
- U19 pad 7: unconnected-(U19-A5-Pad7) -> (no net)
- U19 pad 8: unconnected-(U19-A6-Pad8) -> (no net)
- U19 pad 9: unconnected-(U19-A7-Pad9) -> (no net)
- U20 pad 12: unconnected-(U20-B1-Pad12) -> (no net)
- U20 pad 13: unconnected-(U20-B2-Pad13) -> (no net)
- U20 pad 14: unconnected-(U20-B3-Pad14) -> (no net)
- U20 pad 15: unconnected-(U20-B4-Pad15) -> (no net)
- U20 pad 16: unconnected-(U20-B5-Pad16) -> (no net)
- U20 pad 17: unconnected-(U20-B6-Pad17) -> (no net)
- U20 pad 18: unconnected-(U20-B7-Pad18) -> (no net)
- U4 pad 1: Z_AS -> +5V
- U4 pad 12: Z_OE -> S100_ADSB
- U4 pad 2: Z_DS -> +5V
- U4 pad 25: SLAVE_ONLY -> S100_SDSB
- U4 pad 28: LA1 -> S100_CDSB
- U4 pad 29: LA2 -> SLAVE_WIN
- U4 pad 64: LATCH_LE -> S100_A_OE
- U4 pad 65: SRAM_A0 -> S100_S_OE
- U4 pad 67: SRAM_A1 -> S100_C_OE
- U4 pad 69: MASTER_ACTIVE -> MST_RD
- U4 pad 70: MASTER_WRITE -> MST_WR
- U4 pad 73: BYTE_SEL -> SPLIT
- U4 pad 75: (no net) -> CFG_OE
- U4 pad 76: (no net) -> FLASH_WE
- U4 pad 77: (no net) -> Z_AS
- U4 pad 79: (no net) -> Z_DS
- U4 pad 80: (no net) -> SLV_RD
- U4 pad 81: (no net) -> SLV_WR
- U4 pad 84: (no net) -> +5V
- U5 pad 1: SLAVE -> +5V
- U5 pad 10: A22 -> MST_WR
- U5 pad 11: A23 -> SLV_RD
- U5 pad 12: MASTER_ACTIVE -> SLV_WR
- U5 pad 15: MASTER_WRITE -> XFR16
- U5 pad 16: BYTE_SEL -> SPLIT
- U5 pad 17: XFR16 -> SLAVE
- U5 pad 18: S100_sMEMR -> LA0
- U5 pad 2: A16 -> +5V
- U5 pad 20: S100_sWO -> A0
- U5 pad 21: S100_sXTRQ -> A1
- U5 pad 22: S100_ADSB -> A2
- U5 pad 24: S100_DODSB -> A3
- U5 pad 25: S100_SDSB -> A4
- U5 pad 27: S100_CDSB -> A5
- U5 pad 28: AD0 -> A6
- U5 pad 29: AD1 -> A7
- U5 pad 30: AD2 -> A8
- U5 pad 31: AD3 -> A9
- U5 pad 33: AD4 -> A10
- U5 pad 34: AD5 -> A11
- U5 pad 35: AD6 -> A12
- U5 pad 36: AD7 -> A13
- U5 pad 37: AD8 -> A14
- U5 pad 39: AD9 -> A15
- U5 pad 4: A17 -> Z_AS
- U5 pad 40: AD10 -> AD0
- U5 pad 41: AD11 -> AD1
- U5 pad 44: AD12 -> AD2
- U5 pad 45: AD13 -> AD3
- U5 pad 46: AD14 -> AD4
- U5 pad 48: AD15 -> AD5
- U5 pad 49: S100_DO0 -> AD6
- U5 pad 5: A18 -> Z_DS
- U5 pad 50: S100_DO1 -> AD7
- U5 pad 51: S100_DO2 -> AD8
- U5 pad 52: S100_DO3 -> AD9
- U5 pad 54: S100_DO4 -> AD10
- U5 pad 55: S100_DO5 -> AD11
- U5 pad 56: S100_DO6 -> AD12
- U5 pad 57: S100_DO7 -> AD13
- U5 pad 58: S100_DI0 -> AD14
- U5 pad 6: A19 -> S100_DIR
- U5 pad 60: S100_DI1 -> AD15
- U5 pad 61: S100_DI2 -> S100_DO0
- U5 pad 63: S100_DI3 -> S100_DO1
- U5 pad 64: S100_DI4 -> S100_DO2
- U5 pad 65: S100_DI5 -> S100_DO3
- U5 pad 67: S100_DI6 -> S100_DO4
- U5 pad 68: S100_DI7 -> S100_DO5
- U5 pad 69: SRAM_WIN -> S100_DO6
- U5 pad 70: FLASH_WIN -> S100_DO7
- U5 pad 73: BANK -> S100_DI0
- U5 pad 74: S100_A_OE -> S100_DI1
- U5 pad 75: S100_A_DIR -> S100_DI2
- U5 pad 76: S100_S_OE -> S100_DI3
- U5 pad 77: S100_C_OE -> S100_DI4
- U5 pad 79: S100_SC_DIR -> S100_DI5
- U5 pad 8: A20 -> S100_DODSB
- U5 pad 80: S100_pRDY -> S100_DI6
- U5 pad 81: S100_XRDY -> S100_DI7
- U5 pad 83: S100_SIXTN -> Z_CLK
- U5 pad 84: (no net) -> +5V
- U5 pad 9: A21 -> MST_RD
- U6 pad 1: LA15 -> A15
- U6 pad 10: SRAM_A0 -> A1
- U6 pad 2: LA13 -> A13
- U6 pad 21: LA11 -> A11
- U6 pad 23: LA12 -> A12
- U6 pad 24: LA10 -> A10
- U6 pad 25: LA9 -> A9
- U6 pad 26: LA14 -> A14
- U6 pad 3: LA8 -> A8
- U6 pad 4: LA7 -> A7
- U6 pad 5: LA6 -> A6
- U6 pad 6: LA5 -> A5
- U6 pad 7: LA4 -> A4
- U6 pad 8: LA3 -> A3
- U6 pad 9: SRAM_A1 -> A2
- U7 pad 1: LA15 -> A15
- U7 pad 10: SRAM_A0 -> A1
- U7 pad 2: LA13 -> A13
- U7 pad 21: LA11 -> A11
- U7 pad 23: LA12 -> A12
- U7 pad 24: LA10 -> A10
- U7 pad 25: LA9 -> A9
- U7 pad 26: LA14 -> A14
- U7 pad 3: LA8 -> A8
- U7 pad 4: LA7 -> A7
- U7 pad 5: LA6 -> A6
- U7 pad 6: LA5 -> A5
- U7 pad 7: LA4 -> A4
- U7 pad 8: LA3 -> A3
- U7 pad 9: SRAM_A1 -> A2
- U8 pad 1: LA15 -> A15
- U8 pad 10: SRAM_A0 -> A1
- U8 pad 2: LA13 -> A13
- U8 pad 21: LA11 -> A11
- U8 pad 23: LA12 -> A12
- U8 pad 24: LA10 -> A10
- U8 pad 25: LA9 -> A9
- U8 pad 26: LA14 -> A14
- U8 pad 3: LA8 -> A8
- U8 pad 4: LA7 -> A7
- U8 pad 5: LA6 -> A6
- U8 pad 6: LA5 -> A5
- U8 pad 7: LA4 -> A4
- U8 pad 8: LA3 -> A3
- U8 pad 9: SRAM_A1 -> A2
- U9 pad 1: LA15 -> A15
- U9 pad 10: SRAM_A0 -> A1
- U9 pad 2: LA13 -> A13
- U9 pad 21: LA11 -> A11
- U9 pad 23: LA12 -> A12
- U9 pad 24: LA10 -> A10
- U9 pad 25: LA9 -> A9
- U9 pad 26: LA14 -> A14
- U9 pad 3: LA8 -> A8
- U9 pad 4: LA7 -> A7
- U9 pad 5: LA6 -> A6
- U9 pad 6: LA5 -> A5
- U9 pad 7: LA4 -> A4
- U9 pad 8: LA3 -> A3
- U9 pad 9: SRAM_A1 -> A2
Routing:
- net unconnected-(J8-NC-Pad71): vias 1 -> 0
- net unconnected-(J8-NC-Pad69): vias 1 -> 0
- net unconnected-(J8-NC-Pad66): vias 1 -> 0
- net unconnected-(J8-NC-Pad65): vias 1 -> 0
- net unconnected-(J8-NC-Pad28): vias 1 -> 0
- net unconnected-(J8-NC-Pad27): vias 1 -> 0
- net unconnected-(J8-NC-Pad21): vias 1 -> 0

Commit message: Config straps: consolidate 8x 3-pin jumpers into one 3x8 header
Replace J10-J17 (eight PinHeader_1x03) with a single 24-pin 3x8 header
(J10): one row per BTI bit, col 0 = +5V, col 1 = BTI_ADn, col 2 = GND.
Adds a JP3x8 schematic symbol and a hdr_3x8_fp PCB footprint (pin 1
top-left, row-major, matching the symbol), regenerates the netlist and
board. DRC clean (0 shorting items).

Co-Authored-By: Claude <noreply@anthropic.com>
Parts:
- removed J11: BTI AD1, HDR-3
- removed J12: BTI AD2, HDR-3
- removed J13: BTI AD3, HDR-3
- removed J14: BTI AD4, HDR-3
- removed J15: BTI AD5, HDR-3
- removed J16: BTI AD6, HDR-3
- removed J17: BTI AD7, HDR-3
- J10: value BTI AD0 -> Config (3x8); footprint HDR-3 -> HDR-3x8
- moved J10 33.1 mm to (218.0, 110.0), turned to 90 degrees

Commit message: Z280 S-100: buffer data bus (74F245), move A3-A15 latch out to 74HC573
The ATF1508 macrocell outputs can't meet the IEEE-696 24 mA data-bus sink
spec, so DO0-7 / DI0-7 now run through two 74F245 transceivers (64 mA sink).
DO_DIR / DI_DIR from the data CPLD drive their DIR pins; /OE is tied low
(a 245 in receive mode never drives the bus, so only DIR has to be right),
and both DIRs are DODSB-gated so a temporary master can float the drivers.

To free the two CPLD pins for those DIRs, the plain A3-A15 half of the
address demux latch moved back out to two 74HC573s (LATCH_LE = ~AS, /OE =
SLAVE); A0 (byte lane) and A1/A2 (burst counter) stay in the CPLD. The data
CPLD now fits at 53/64 I/O (was 64/64).

Also: the address 245s referenced stale LA1-15 nets while the CPLD drove
A1-15, leaving S-100 A1-A15 floating -- fixed. The redundant S100_DIR output
is gone; address/status/control 245 DIR is now wired straight to Z_BUSACK.

Co-Authored-By: Claude Code <noreply@anthropic.com>
Parts:
- added C20: 0.1uF, CAP-2, F.Cu at (162.0, 68.0)
- added C21: 0.1uF, CAP-2, F.Cu at (174.0, 68.0)
- added C22: 0.1uF, CAP-2, F.Cu at (186.0, 68.0)
- added C23: 0.1uF, CAP-2, F.Cu at (198.0, 68.0)
- added U2: 74HC573 latch, DIP-20, F.Cu at (162.0, 50.0)
- added U25: 74F245 DO, DIP-20, F.Cu at (186.0, 50.0)
- added U26: 74F245 DI, DIP-20, F.Cu at (198.0, 50.0)
- added U3: 74HC573 latch, DIP-20, F.Cu at (174.0, 50.0)
- moved C17 40.2 mm to (142.0, 67.0)
- moved C16 35.7 mm to (130.0, 67.0)
Connections:
- U15 pad 1: S100_DIR -> Z_BUSACK
- U15 pad 3: LA1 -> A1
- U15 pad 4: LA2 -> A2
- U15 pad 5: LA3 -> A3
- U15 pad 6: LA4 -> A4
- U15 pad 7: LA5 -> A5
- U15 pad 8: LA6 -> A6
- U15 pad 9: LA7 -> A7
- U16 pad 1: S100_DIR -> Z_BUSACK
- U16 pad 2: LA8 -> A8
- U16 pad 3: LA9 -> A9
- U16 pad 4: LA10 -> A10
- U16 pad 5: LA11 -> A11
- U16 pad 6: LA12 -> A12
- U16 pad 7: LA13 -> A13
- U16 pad 8: LA14 -> A14
- U16 pad 9: LA15 -> A15
- U17 pad 1: S100_DIR -> Z_BUSACK
- U18 pad 1: S100_DIR -> Z_BUSACK
- U19 pad 1: S100_DIR -> Z_BUSACK
- U5 pad 24: A3 -> DO_DIR
- U5 pad 25: A4 -> DI_DIR
- U5 pad 27: A5 -> (no net)
- U5 pad 28: A6 -> (no net)
- U5 pad 29: A7 -> (no net)
- U5 pad 30: A8 -> (no net)
- U5 pad 31: A9 -> (no net)
- U5 pad 33: A10 -> (no net)
- U5 pad 34: A11 -> (no net)
- U5 pad 35: A12 -> (no net)
- U5 pad 36: A13 -> (no net)
- U5 pad 37: A14 -> (no net)
- U5 pad 39: A15 -> (no net)
- U5 pad 6: S100_DIR -> LATCH_LE
- U5 pad 61: S100_DO0 -> CPLD_DO0
- U5 pad 63: S100_DO1 -> CPLD_DO1
- U5 pad 64: S100_DO2 -> CPLD_DO2
- U5 pad 65: S100_DO3 -> CPLD_DO3
- U5 pad 67: S100_DO4 -> CPLD_DO4
- U5 pad 68: S100_DO5 -> CPLD_DO5
- U5 pad 69: S100_DO6 -> CPLD_DO6
- U5 pad 70: S100_DO7 -> CPLD_DO7
- U5 pad 73: S100_DI0 -> CPLD_DI0
- U5 pad 74: S100_DI1 -> CPLD_DI1
- U5 pad 75: S100_DI2 -> CPLD_DI2
- U5 pad 76: S100_DI3 -> CPLD_DI3
- U5 pad 77: S100_DI4 -> CPLD_DI4
- U5 pad 79: S100_DI5 -> CPLD_DI5
- U5 pad 80: S100_DI6 -> CPLD_DI6
- U5 pad 81: S100_DI7 -> CPLD_DI7
