File: z280-s100.kicad_pcb (KiCad board)
At the start: 4 copper layers, 254 x 134.6 mm, 60 parts, among them J10 Config header (3x8), J7 Serial header (2x5), J8 S-100, J9 JTAG header (1x6), U1 Z280 Z-BUS, U10 AT28C256 HI, U11 AT28C256 LO, U12 LM7805, U13 DS1813, U14 MAX232, U15 74HCT245, U16 74HCT245, U17 74HCT245, U18 74HCT245, U19 74HCT245, U2 74HC573, U20 74HCT245, U21 74HCT244, U22 74F138, U23 74F521, U24 74F521, U25 74F245, U26 74F245, U27 LM323K, U3 74HC573, U4 ATF1508AS (PLCC-84), U5 ATF1508AS (PLCC-84), U6 RAM0 HI, U7 RAM0 LO, U8 RAM1 HI, U9 RAM1 LO, Y1 24 MHz, Y2 24 MHz

Commit message: Z280 S-100: CPLD pin re-site, SLAVE_ONLY strap, full route + patch area
- Re-pin both CPLDs so signals sit on the package side facing their
  consumers (memory enables up, Z-BUS left, steering right, S-100
  status/control down).
- Restore SLAVE_ONLY debug strap (arbitration: SLAVE = !Z_BUSACK #
  SLAVE_ONLY) + J11 2-pin header + R3 1k pull-down.
- Move interrupts (S100_INT/NMI, Z_INT/Z_NMI) to the data CPLD to free
  control-CPLD pins.
- gen_pcb.py now regenerates the board ab initio: S-100 test-point vias +
  finger traces cloned verbatim, U27 LM323K, +8V island, power planes,
  J11 header, and a 16x10 patch area (PTH sea of holes, 0.1" pitch,
  0.8 mm drills) clear of the DI bus in the upper-right.
- Full FreeRouting pass (2-layer lie workflow, via_costs=15): signal nets
  routed on F.Cu/B.Cu with planes kept off the outer layers; S100_DI2 and
  S100_NMI left hand-routed.

Co-Authored-By: Claude Code <noreply@anthropic.com>
Parts:
- removed Y2: 24 MHz, z280-s100:Oscillator_DIP-8-14
- added ?: , PATCH, F.Cu at (226.0, 116.0)
- added J11: SLAVE_ONLY jumper, Connector_PinHeader_2.54mm:PinHeader_1x02_P2.54mm_Vertical, F.Cu at (250.0, 51.3)
- C14, C15: moved to F.Cu
- J10: value Config header (3x8) -> Config (3x8)
- J7: value Serial header (2x5) -> Serial (2x5)
- J8: value S-100 -> S-100 edge
- J9: value JTAG header (1x6) -> JTAG (1x6); footprint Connector_PinHeader_2.54mm:PinHeader_1x06_P2.54mm_Vertical -> HDR-6
- R1: value 1k -> 1k pRDY; footprint Resistor_THT:R_Axial_DIN0207_L6.3mm_D2.5mm_P7.62mm_Horizontal -> HDR-2
- R2: value 1k -> 1k XRDY; footprint Resistor_THT:R_Axial_DIN0207_L6.3mm_D2.5mm_P7.62mm_Horizontal -> HDR-2
- R3: value 1k -> 1k SLAVE_ONLY; footprint Resistor_THT:R_Axial_DIN0207_L6.3mm_D2.5mm_P7.62mm_Horizontal -> HDR-2
- R4: value 1k -> 1k SIXTN; footprint Resistor_THT:R_Axial_DIN0207_L6.3mm_D2.5mm_P7.62mm_Horizontal -> HDR-2
- U1: value Z280 Z-BUS -> Z280 (PLCC-68)
- U10: value AT28C256 HI -> 28C256 even
- U11: value AT28C256 LO -> 28C256 odd
- U12: value LM7805 -> 7805; footprint Package_TO_SOT_THT:TO-220-3_Horizontal_TabDown -> HDR-3
- U13: value DS1813 -> DS1813 reset; footprint Package_TO_SOT_THT:TO-92_Inline -> HDR-3
- U15: value 74HCT245 -> 74HCT245 addr0
- U16: value 74HCT245 -> 74HCT245 addr1
- U17: value 74HCT245 -> 74HCT245 addr2
- U18: value 74HCT245 -> 74HCT245 status
- U19: value 74HCT245 -> 74HCT245 control
- U2, U3: value 74HC573 -> 74HC573 latch
- U20: value 74HCT245 -> 74HCT245 pHLDA
- U21: value 74HCT244 -> 74HCT244 BTI
- U22: value 74F138 -> 74F138 decode
- U23: value 74F521 -> 74F521 flash win
- U24: value 74F521 -> 74F521 slave win
- U25: value 74F245 -> 74F245 DO
- U26: value 74F245 -> 74F245 DI
- U4: value ATF1508AS (PLCC-84) -> ATF1508 control
- U5: value ATF1508AS (PLCC-84) -> ATF1508 data
- U6: value RAM0 HI -> SRAM bank0 even
- U7: value RAM0 LO -> SRAM bank0 odd
- U8: value RAM1 HI -> SRAM bank1 even
- U9: value RAM1 LO -> SRAM bank1 odd
- Y1: value 24 MHz -> 24 MHz crystal
- moved U12 3.97 mm to (22.7, 139.2)
- turned C14 to 0 degrees
- turned C15 to 0 degrees
- turned C16 to 0 degrees
- turned C17 to 0 degrees
Connections:
- U4 pad 10: Z_ST3 -> MEM_CE0
- U4 pad 11: Z_IE -> CFG_OE
- U4 pad 12: S100_ADSB -> Z_AS
- U4 pad 15: Z_BUSACK -> Z_DS
- U4 pad 16: Z_RESET -> Z_RW
- U4 pad 17: S100_INT -> Z_BW
- U4 pad 18: S100_NMI -> Z_ST0
- U4 pad 20: S100_HOLD -> Z_ST1
- U4 pad 21: S100_pRDY -> Z_ST2
- U4 pad 22: S100_XRDY -> Z_ST3
- U4 pad 24: S100_SIXTN -> Z_IE
- U4 pad 25: S100_SDSB -> Z_BUSACK
- U4 pad 27: LA0 -> Z_RESET
- U4 pad 28: S100_CDSB -> Z_WAIT
- U4 pad 29: SLAVE_WIN -> Z_BUSREQ
- U4 pad 30: SRAM_WIN -> CPLD_sINTA
- U4 pad 31: FLASH_WIN -> CPLD_sHLTA
- U4 pad 33: A20 -> S100_HOLD
- U4 pad 34: Z_WAIT -> S100_pRDY
- U4 pad 35: Z_INT -> S100_XRDY
- U4 pad 36: Z_NMI -> S100_ADSB
- U4 pad 37: Z_BUSREQ -> S100_SDSB
- U4 pad 39: CPLD_sMEMR -> S100_CDSB
- U4 pad 4: Z_RW -> MEM_WE_H
- U4 pad 40: CPLD_sWO -> S100_SIXTN
- U4 pad 41: CPLD_sINP -> CPLD_pSYNC
- U4 pad 44: CPLD_sOUT -> CPLD_pSTVAL
- U4 pad 45: CPLD_sINTA -> CPLD_pDBIN
- U4 pad 46: CPLD_sHLTA -> CPLD_pWR
- U4 pad 48: CPLD_sXTRQ -> CPLD_pHLDA
- U4 pad 49: CPLD_pSYNC -> CPLD_sMEMR
- U4 pad 5: Z_BW -> MEM_OE
- U4 pad 50: CPLD_pSTVAL -> CPLD_sWO
- U4 pad 51: CPLD_pDBIN -> CPLD_sINP
- U4 pad 52: CPLD_pWR -> CPLD_sOUT
- U4 pad 54: CPLD_pHLDA -> MST_RD
- U4 pad 55: MEM_CE0 -> MST_WR
- U4 pad 56: MEM_CE1 -> SLV_RD
- U4 pad 57: MEM_OE -> SLV_WR
- U4 pad 58: MEM_WE_L -> SLAVE
- U4 pad 6: Z_ST0 -> MEM_WE_L
- U4 pad 60: MEM_WE_H -> XFR16
- U4 pad 61: FLASH_CE -> SPLIT
- U4 pad 63: FLASH_OE -> LA0
- U4 pad 64: S100_A_OE -> SLAVE_ONLY
- U4 pad 65: S100_S_OE -> CPLD_sXTRQ
- U4 pad 67: S100_C_OE -> S100_A_OE
- U4 pad 68: SLAVE -> S100_S_OE
- U4 pad 69: MST_RD -> S100_C_OE
- U4 pad 70: MST_WR -> SRAM_WIN
- U4 pad 73: SPLIT -> FLASH_WIN
- U4 pad 74: XFR16 -> SLAVE_WIN
- U4 pad 75: CFG_OE -> (no net)
- U4 pad 76: FLASH_WE -> (no net)
- U4 pad 77: Z_AS -> (no net)
- U4 pad 79: Z_DS -> FLASH_OE
- U4 pad 8: Z_ST1 -> MEM_CE1
- U4 pad 80: SLV_RD -> FLASH_WE
- U4 pad 81: SLV_WR -> FLASH_CE
- U4 pad 9: Z_ST2 -> A20
- U5 pad 10: MST_WR -> AD8
- U5 pad 11: SLV_RD -> AD9
- U5 pad 12: SLV_WR -> MST_RD
- U5 pad 15: XFR16 -> MST_WR
- U5 pad 16: SPLIT -> SLV_RD
- U5 pad 17: SLAVE -> SLV_WR
- U5 pad 18: LA0 -> XFR16
- U5 pad 20: A0 -> SPLIT
- U5 pad 21: A1 -> SLAVE
- U5 pad 22: A2 -> LA0
- U5 pad 24: DO_DIR -> AD0
- U5 pad 25: DI_DIR -> AD1
- U5 pad 27: (no net) -> AD2
- U5 pad 28: (no net) -> AD3
- U5 pad 29: (no net) -> AD4
- U5 pad 30: (no net) -> AD5
- U5 pad 31: (no net) -> AD6
- U5 pad 33: (no net) -> CPLD_DO0
- U5 pad 34: (no net) -> CPLD_DO1
- U5 pad 35: (no net) -> CPLD_DO2
- U5 pad 36: (no net) -> CPLD_DO3
- U5 pad 37: (no net) -> CPLD_DO4
- U5 pad 39: (no net) -> CPLD_DO5
- U5 pad 4: Z_AS -> A0
- U5 pad 40: AD0 -> CPLD_DO6
- U5 pad 41: AD1 -> CPLD_DO7
- U5 pad 44: AD2 -> CPLD_DI0
- U5 pad 45: AD3 -> CPLD_DI1
- U5 pad 46: AD4 -> CPLD_DI2
- U5 pad 48: AD5 -> CPLD_DI3
- U5 pad 49: AD6 -> CPLD_DI4
- U5 pad 5: Z_DS -> A1
- U5 pad 50: AD7 -> CPLD_DI5
- U5 pad 51: AD8 -> CPLD_DI6
- U5 pad 52: AD9 -> CPLD_DI7
- U5 pad 54: AD10 -> Z_AS
- U5 pad 55: AD11 -> Z_DS
- U5 pad 56: AD12 -> Z_INT
- U5 pad 57: AD13 -> Z_NMI
- U5 pad 58: AD14 -> DO_DIR
- U5 pad 6: LATCH_LE -> A2
- U5 pad 60: AD15 -> DI_DIR
- U5 pad 61: CPLD_DO0 -> S100_DODSB
- U5 pad 63: CPLD_DO1 -> S100_INT
- U5 pad 64: CPLD_DO2 -> S100_NMI
- U5 pad 65: CPLD_DO3 -> (no net)
- U5 pad 67: CPLD_DO4 -> (no net)
- U5 pad 68: CPLD_DO5 -> (no net)
- U5 pad 69: CPLD_DO6 -> (no net)
- U5 pad 70: CPLD_DO7 -> (no net)
- U5 pad 73: CPLD_DI0 -> (no net)
- U5 pad 74: CPLD_DI1 -> (no net)
- U5 pad 75: CPLD_DI2 -> AD10
- U5 pad 76: CPLD_DI3 -> AD11
- U5 pad 77: CPLD_DI4 -> AD12
- U5 pad 79: CPLD_DI5 -> AD13
- U5 pad 8: S100_DODSB -> LATCH_LE
- U5 pad 80: CPLD_DI6 -> AD14
- U5 pad 81: CPLD_DI7 -> AD15
- U5 pad 9: MST_RD -> AD7
Routing:
- net A7: track 0.00 -> 292.0 mm, vias 0 -> 2
- net AD4: track 0.00 -> 284.7 mm, vias 0 -> 7
- net AD5: track 0.00 -> 283.9 mm, vias 0 -> 5
- net AD6: track 0.00 -> 276.4 mm, vias 0 -> 7
- net AD7: track 0.00 -> 275.6 mm, vias 0 -> 6
- net AD1: track 0.00 -> 274.8 mm, vias 0 -> 8
- net AD3: track 0.00 -> 274.0 mm, vias 0 -> 3
- net AD2: track 0.00 -> 270.8 mm, vias 0 -> 4
- net A2: track 0.00 -> 265.8 mm, vias 0 -> 2
- net A13: track 0.00 -> 263.1 mm, vias 0 -> 3
- net A6: track 0.00 -> 261.5 mm, vias 0 -> 1
- net A15: track 0.00 -> 260.9 mm
- net A14: track 0.00 -> 259.4 mm, vias 0 -> 3
- net AD0: track 0.00 -> 257.4 mm, vias 0 -> 2
- net A5: track 0.00 -> 255.9 mm, vias 0 -> 2
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