File: z280-s100.kicad_pcb (KiCad board)
At the start: 4 copper layers, 254 x 134.6 mm, 61 parts, among them J10 Config (3x8), J11 SLAVE_ONLY jumper, J7 Serial (2x5), J8 S-100 edge, J9 JTAG (1x6), U1 Z280 (PLCC-68), U10 28C256 even, U11 28C256 odd, U12 7805, U13 DS1813 reset, U14 MAX232, U15 74HCT245 addr0, U16 74HCT245 addr1, U17 74HCT245 addr2, U18 74HCT245 status, U19 74HCT245 control, U2 74HC573 latch, U20 74HCT245 pHLDA, U21 74HCT244 BTI, U22 74F138 decode, U23 74F521 flash win, U24 74F521 slave win, U25 74F245 DO, U26 74F245 DI, U27 LM323K, U3 74HC573 latch, U4 ATF1508 control, U5 ATF1508 data, U6 SRAM bank0 even, U7 SRAM bank0 odd, U8 SRAM bank1 even, U9 SRAM bank1 odd, Y1 24 MHz crystal

Commit message: Z280 S-100: relabel 74F bus parts, silk values, CPLD JEDECs + pin docs
- Address/status/control drivers 74HCT245 -> 74F245; address latch 74HC573 ->
  74F573. 74ACT245/74ACT573 are documented drop-in substitutes at build time
  if the F parts draw too much +5V.
- Move footprint Value from F.Fab to F.SilkS and strip the descriptive
  suffixes so the silkscreen matches the hand-edited board (74F245, 74F573,
  74F138, ...). F.Fab stays a comment-only layer.
- Generate ATF1508 JEDECs for the re-sited CPLDs (ad: 53 MC/3 FF, ctl: 43 MC/7
  FF; pin assignments kept). Document unused I/O for a board rev 2: U5 has
  65/67/68/69/70/73/74 free, U4 has 75/76/77 free + Z_AS (pin 12) as a spare.

Co-Authored-By: Claude Code <noreply@anthropic.com>
Parts:
- J10: value Config (3x8) -> Config
- J11: value SLAVE_ONLY jumper -> SLAVE_ONLY
- J9: value JTAG (1x6) -> JTAG
- U1: value Z280 (PLCC-68) -> Z280 (ZBUS)
- U13: value DS1813 reset -> DS1813
- U15: value 74HCT245 addr0 -> 74F245
- U16: value 74HCT245 addr1 -> 74F245
- U17: value 74HCT245 addr2 -> 74F245
- U18: value 74HCT245 status -> 74F245
- U19: value 74HCT245 control -> 74F245
- U2, U3: value 74HC573 latch -> 74F573
- U20: value 74HCT245 pHLDA -> 74F245
- U21: value 74HCT244 BTI -> 74HCT244
- U22: value 74F138 decode -> 74F138
- U23: value 74F521 flash win -> 74F521
- U24: value 74F521 slave win -> 74F521
- U25: value 74F245 DO -> 74F245
- U26: value 74F245 DI -> 74F245
- U6: value SRAM bank0 even -> SRAM0 even
- U7: value SRAM bank0 odd -> SRAM0 odd
- U8: value SRAM bank1 even -> SRAM1 even
- U9: value SRAM bank1 odd -> SRAM1 odd
- V 0.1 curt@zen-room.org: renamed from J8; value S-100 edge -> Z280 16 Bit Master
Routing:
- net A7: track 292.0 -> 281.2 mm
