File: z280-s100.kicad_sch (KiCad schematic)
At the start: 43 parts, among them J10 Config header (3x8), J11 Jumper (2-pin header), J7 Serial header (2x5), J8 S-100 edge connector (100-pin), J9 JTAG header (1x6), U1 Z280 Z-BUS (12 MHz), U10 AT28C256 (32Kx8), U11 AT28C256 (32Kx8), U12 LM7805, U13 DS1813, U14 MAX232, U15 74F245, U16 74F245, U17 74F245, U18 74F245, U19 74F245, U2 74F573, U20 74F245, U21 74HCT244, U22 74F138, U23 74F521, U24 74F521, U25 74F245, U26 74F245, U27 LM323K, U3 74F573, U4 ATF1508AS (PLCC-84), U5 ATF1508AS (PLCC-84), U6 IS61C5128AS-25QLI (512Kx8), U7 IS61C5128AS-25QLI (512Kx8), U8 IS61C5128AS-25QLI (512Kx8), U9 IS61C5128AS-25QLI (512Kx8), Y1 24 MHz, Y2 24 MHz

Commit message: V2.0 rev 3: 4 MB RAM, boot ROM at 400000 + overlay, W window register
- RAM grows to 4 MB (8x IS61C5128AS-25), bank select off-chip via 74F139
  (RAM_SELECT enable + A1_EFF:A20 = Z_OWN ? A21:A20 : W:A20)
- boot ROM moves to 400000; control CPLD aliases it at 0 until the first
  memory write clears BOOTED (bootrom.s sketches the boot sequence)
- W: 1-bit window register, settable locally (register block Y3/Y4) and over
  S-100 (doorbell ports 100/101), held in the doorbell GAL
- doorbell widens 4->8 ports (A2:A0), range base 6->5 bits
- SLAVE_WIN back to a 2 MB window; FLASH_WIN 0xF0->0x40

Co-Authored-By: Claude Code <noreply@anthropic.com>
Parts:
- added J12, J13, J14, J15, J16: Jumper (3-pin header), Connector_PinHeader_2.54mm:PinHeader_1x03_P2.54mm_Vertical, symbol z280s100:JP3
- added R5: 1k, Resistor_THT:R_Axial_DIN0207_L6.3mm_D2.5mm_P7.62mm_Horizontal, symbol z280s100:R
- added U28, U32: 74F521, Package_DIP:DIP-20_W7.62mm, symbol z280s100:74F521
- added U29: ATF22V10 (doorbell), Package_DIP:DIP-24_W15.24mm, symbol z280s100:DOORBELL
- added U30, U31: 74F574, Package_DIP:DIP-20_W7.62mm, symbol z280s100:74F574
- added U33: 74F138, Package_DIP:DIP-16_W7.62mm, symbol z280s100:74F138
- added U34, U35: 74HCT244, Package_DIP:DIP-20_W7.62mm, symbol z280s100:74HCT244
- added U36, U37, U38, U39: IS61C5128AS-25QLI (512Kx8), Package_DIP:DIP-32_W15.24mm, symbol z280s100:IS61C5128AS
- added U40: 74F139, Package_DIP:DIP-16_W7.62mm, symbol z280s100:74F139
- U13: value DS1813 -> MAX708; footprint Package_TO_SOT_THT:TO-92_Inline -> Package_DIP:DIP-8_W7.62mm; symbol z280s100:DS1813 -> z280s100:MAX708
Connections:
- net A0 is gone; now on net +5V: U15.2 (A0), U5.4 (A0)
- net A1 is gone; now on net +5V: U10.10 (A0), U11.10 (A0), U15.3 (A1), U5.5 (A1), U6.12 (A0), U7.12 (A0), U8.12 (A0), U9.12 (A0)
- net A11 is gone; now on net +5V: U10.21 (A10), U11.21 (A10), U16.5 (A3), U3.12 (Q0), U6.23 (A10), U7.23 (A10), U8.23 (A10), U9.23 (A10)
- net A13 is gone; now on net +5V: U10.2 (A12), U11.2 (A12), U16.7 (A5), U3.14 (Q2), U6.4 (A12), U7.4 (A12), U8.4 (A12), U9.4 (A12)
- net A16 is gone; now on net +5V: U1.5 (A16), U17.2 (A0), U23.3 (Q0), U24.2 (P0), U24.3 (Q0), U6.31 (A15), U7.31 (A15), U8.31 (A15), U9.31 (A15)
- net A17 is gone; now on net +5V: U1.6 (A17), U17.3 (A1), U23.5 (Q1), U24.4 (P1), U24.5 (Q1), U6.2 (A16), U7.2 (A16), U8.2 (A16), U9.2 (A16)
- net A18 is gone; now on net +5V: U1.8 (A18), U17.4 (A2), U23.7 (Q2), U24.6 (P2), U24.7 (Q2), U6.1 (A17), U7.1 (A17), U8.1 (A17), U9.1 (A17)
- net A2 is gone; now on net +5V: U10.9 (A1), U11.9 (A1), U15.4 (A2), U5.6 (A2), U6.11 (A1), U7.11 (A1), U8.11 (A1), U9.11 (A1)
- net A22 is gone; now on net +5V: U1.66 (A22), U17.8 (A6), U22.2 (A1), U23.15 (Q6), U24.15 (Q6)
- net A3 is gone; now on net +5V: U10.8 (A2), U11.8 (A2), U15.5 (A3), U2.12 (Q0), U6.10 (A2), U7.10 (A2), U8.10 (A2), U9.10 (A2)
- net A4 is gone; now on net +5V: U10.7 (A3), U11.7 (A3), U15.6 (A4), U2.13 (Q1), U6.9 (A3), U7.9 (A3), U8.9 (A3), U9.9 (A3)
- net A5 is gone; now on net +5V: U10.6 (A4), U11.6 (A4), U15.7 (A5), U2.14 (Q2), U6.8 (A4), U7.8 (A4), U8.8 (A4), U9.8 (A4)
- net A9 is gone; now on net A7: U10.25 (A8), U11.25 (A8), U16.3 (A1), U2.18 (Q6), U6.27 (A8), U7.27 (A8), U8.27 (A8), U9.27 (A8)
- net AD1 is gone; now on net +5V: U1.42 (AD1), U11.12 (DQ1), U21.16 (Y1), U5.25 (AD1), U7.14 (DQ1), U9.14 (DQ1)
- net AD10 is gone; now on net +5V: U1.65 (AD10), U10.13 (DQ2), U2.9 (D7), U5.75 (AD10), U6.15 (DQ2), U8.15 (DQ2)
- net AD13 is gone; now on net +5V: U1.2 (AD13), U10.17 (DQ5), U3.4 (D2), U5.79 (AD13), U6.19 (DQ5), U8.19 (DQ5)
- net AD15 is gone; now on net +5V: U1.4 (AD15), U10.19 (DQ7), U3.6 (D4), U5.81 (AD15), U6.21 (DQ7), U8.21 (DQ7)
- net AD2 is gone; now on net A21: U1.43 (AD2), U11.13 (DQ2), U21.14 (Y2), U5.27 (AD2), U7.15 (DQ2), U9.15 (DQ2)
- net AD3 is gone; now on net +5V: U1.44 (AD3), U11.15 (DQ3), U2.2 (D0), U21.12 (Y3), U5.28 (AD3), U7.17 (DQ3), U9.17 (DQ3)
- net AD8 is gone; now on net +5V: U1.62 (AD8), U10.11 (DQ0), U2.7 (D5), U5.10 (AD8), U6.13 (DQ0), U8.13 (DQ0)
- net AD9 is gone; now on net A21: U1.64 (AD9), U10.12 (DQ1), U2.8 (D6), U5.11 (AD9), U6.14 (DQ1), U8.14 (DQ1)
- net FLASH_CE is gone; now on net +5V: U10.20 (CE), U11.20 (CE), U4.81 (FLASH_CE)
- net FLASH_OE is gone; now on net +5V: U10.22 (OE), U11.22 (OE), U4.79 (FLASH_OE)
- net GND is gone; now on net +5V: C3.2, C4.2, C5.2, J10.12 (LOW), J10.15 (LOW), J10.18 (LOW), J10.21 (LOW), J10.24 (LOW), J10.3 (LOW), J10.6 (LOW), J10.9 (LOW), J7.10 (GND), J7.3 (GND), J7.4 (GND), J7.5 (GND), J7.6 (GND), J7.7 (GND), J7.8 (GND), J7.9 (GND), J8.100 (GND), J8.20 (GND), J8.50 (GND), J8.53 (GND), J8.70 (GND), J9.5 (GND), R3.1, U1.1 (GND), U1.35 (GND), U1.51 (GND), U1.53 (GND), U10.14 (GND), U11.14 (GND), U12.2 (GND), U13.1 (MR), U14.15 (GND), U15.10 (GND), U16.10 (GND), U17.10 (GND), U18.10 (GND), U19.10 (GND), U2.10 (GND), U20.10 (GND), U20.19 (OE), U20.3 (A1), U20.4 (A2), U20.5 (A3), U20.6 (A4), U20.7 (A5), U20.8 (A6), U20.9 (A7), U21.10 (GND), U22.4 (G2A), U22.5 (G2B), U22.8 (GND), U23.1 (G), U23.10 (GND), U23.2 (P0), U23.4 (P1), U23.6 (P2), U23.8 (P3), U24.1 (G), U24.10 (GND), U24.14 (P5), U24.16 (P6), U24.18 (P7), U25.10 (GND), U25.19 (OE), U26.10 (GND), U26.19 (OE), U27.3 (GND), U3.10 (GND), U3.7 (D5), U3.8 (D6), U3.9 (D7), U4.19 (GND), U4.32 (GND), U4.42 (GND), U4.47 (GND), U4.59 (GND), U4.7 (GND), U4.72 (GND), U4.82 (GND), U5.19 (GND), U5.32 (GND), U5.42 (GND), U5.47 (GND), U5.59 (GND), U5.7 (GND), U5.72 (GND), U5.82 (GND), U6.16 (GND), U7.16 (GND), U8.16 (GND), U9.16 (GND), Y2.4 (GND), Y2.7 (GND)
- net JTAG_TCK is gone; now on net AD4: J9.1 (TCK), U4.62 (TCK), U5.62 (TCK)
- net JTAG_TMS is gone; now on net +5V: J9.2 (TMS), U4.23 (TMS), U5.23 (TMS)
- net MST_RD is gone; now on net A6: U4.54 (MST_RD), U5.12 (MST_RD)
- net NC is gone; now on net +5V: U14.10 (T2IN), U14.7 (T2OUT), U14.8 (R2IN), U14.9 (R2OUT)
- net S100_A7 is gone; now on net A6: J8.83 (A7), U15.18 (B7)
- net S100_RESET is gone; now on net +5V: J8.75 (RESET)
- net S100_SLAVE_CLR is gone; now on net +5V: J8.54 (SLAVE_CLR)
- net SLAVE is gone; now on net AD5: U2.1 (OE), U3.1 (OE), U4.58 (SLAVE), U5.21 (SLAVE)
- net SLV_RD is gone; now on net AD7: U4.56 (SLV_RD), U5.16 (SLV_RD)
- net XFR16 is gone; now on net AD6: U4.60 (XFR16), U5.18 (XFR16)
- net Z_RESET is gone; now on net +5V: U1.38 (RESET), U13.2 (VCC), U4.27 (Z_RESET)
- net +5V: now also U1.45 (A20), U13.4 (PFI), U13.5 (PFO), U13.6 (NC), U13.7 (RESET), U17.6 (A4), U22.1 (A0), U23.11 (Q4), U24.11 (Q4), U24.12 (P4), U5.56 (Z_RESET), J12.1 (HIGH), J12.3 (LOW), J13.1 (HIGH), J13.3 (LOW), J14.1 (HIGH), J14.3 (LOW), J15.1 (HIGH), J15.3 (LOW), J16.1 (HIGH), J16.3 (LOW), R5.1, R5.2, U28.1 (G), U28.10 (GND), U28.13 (Q5), U28.14 (P5), U28.15 (Q6), U28.16 (P6), U28.17 (Q7), U28.18 (P7), U28.20 (+5V), U29.11 (LOC_W0), U29.12 (GND), U29.16 (SM_FULL), U29.17 (Z_RST), U29.24 (+5V), U29.7 (Z_RESET), U30.1 (OE), U30.10 (GND), U30.16 (Q4), U30.17 (Q5), U30.18 (Q6), U30.20 (+5V), U31.1 (OE), U31.10 (GND), U31.20 (+5V), U31.3 (D1), U31.5 (D3), U32.1 (G), U32.10 (GND), U32.11 (Q4), U32.12 (P4), U32.13 (Q5), U32.15 (Q6), U32.16 (P6), U32.17 (Q7), U32.2 (P0), U32.20 (+5V), U32.3 (Q0), U32.4 (P1), U32.5 (Q1), U32.6 (P2), U32.7 (Q2), U32.9 (Q3), U33.1 (A0), U33.10 (Y5), U33.12 (Y3), U33.16 (+5V), U33.2 (A1), U33.3 (A2), U33.4 (G2A), U33.5 (G2B), U33.7 (Y7), U33.8 (GND), U33.9 (Y6), U34.10 (GND), U34.11 (A4), U34.12 (Y3), U34.13 (A5), U34.15 (A6), U34.16 (Y1), U34.20 (+5V), U35.10 (GND), U35.16 (Y1), U35.20 (+5V), U35.4 (A1), U36.1 (A17), U36.10 (A2), U36.11 (A1), U36.12 (A0), U36.13 (DQ0), U36.15 (DQ2), U36.16 (GND), U36.19 (DQ5), U36.2 (A16), U36.21 (DQ7), U36.22 (CE), U36.23 (A10), U36.31 (A15), U36.32 (VCC), U36.4 (A12), U36.8 (A4), U36.9 (A3), U37.1 (A17), U37.10 (A2), U37.11 (A1), U37.12 (A0), U37.14 (DQ1), U37.16 (GND), U37.17 (DQ3), U37.2 (A16), U37.22 (CE), U37.23 (A10), U37.31 (A15), U37.32 (VCC), U37.4 (A12), U37.8 (A4), U37.9 (A3), U38.1 (A17), U38.10 (A2), U38.11 (A1), U38.12 (A0), U38.13 (DQ0), U38.15 (DQ2), U38.16 (GND), U38.19 (DQ5), U38.2 (A16), U38.21 (DQ7), U38.22 (CE), U38.23 (A10), U38.31 (A15), U38.32 (VCC), U38.4 (A12), U38.8 (A4), U38.9 (A3), U39.1 (A17), U39.10 (A2), U39.11 (A1), U39.12 (A0), U39.14 (DQ1), U39.16 (GND), U39.17 (DQ3), U39.2 (A16), U39.22 (CE), U39.23 (A10), U39.31 (A15), U39.32 (VCC), U39.4 (A12), U39.8 (A4), U39.9 (A3), U40.11 (Y12), U40.13 (A12), U40.14 (A02), U40.15 (E2), U40.16 (+5V), U40.2 (A01), U40.6 (Y21), U40.7 (Y31), U40.8 (GND)
- net A10: now also U36.26 (A9), U37.26 (A9), U38.26 (A9), U39.26 (A9)
- net A12: now also U36.25 (A11), U37.25 (A11), U38.25 (A11), U39.25 (A11)
- net A14: now also U35.2 (A0), U36.28 (A13), U37.28 (A13), U38.28 (A13), U39.28 (A13)
- net A15: now also U4.10 (RAM_SELECT), U29.13 (LOC_W1), U33.11 (Y4), U36.3 (A14), U37.3 (A14), U38.3 (A14), U39.3 (A14), U40.1 (E1)
- net A19: now also U32.8 (P3), U36.30 (A18), U37.30 (A18), U38.30 (A18), U39.30 (A18)
- net A21: now also U13.8 (RESET), U4.9 (A21), U28.19 (PEQQ), U29.2 (MATCH), U31.4 (D2), U32.14 (P5), U34.14 (Y2), U35.14 (Y2), U36.14 (DQ1), U37.15 (DQ2), U38.14 (DQ1), U39.15 (DQ2); no longer U22.1 (A0)
- net A23: now also U32.18 (P7)
- net A6: now also U8.22 (CE), U9.22 (CE), U28.12 (P4), U29.9 (MS_CLR), U33.15 (Y0), U34.1 (OE1), U34.19 (OE2), U36.7 (A5), U37.7 (A5), U38.7 (A5), U39.7 (A5), U40.5 (Y11)
- net A7: now also U6.22 (CE), U7.22 (CE), J16.2 (SEL), U28.11 (Q4), U33.14 (Y1), U35.1 (OE1), U35.19 (OE2), U36.27 (A8), U36.6 (A6), U37.27 (A8), U37.6 (A6), U38.27 (A8), U38.6 (A6), U39.27 (A8), U39.6 (A6), U40.4 (Y01)
- net AD0: now also U31.2 (D0), U34.18 (Y0), U35.18 (Y0), U37.13 (DQ0), U39.13 (DQ0)
- net AD11: now also U36.17 (DQ3), U38.17 (DQ3), U40.9 (Y32)
- net AD12: now also U36.18 (DQ4), U38.18 (DQ4), U40.10 (Y22)
- net AD14: now also U36.20 (DQ6), U38.20 (DQ6), U40.12 (Y02)
- net AD4: now also U31.6 (D4), U34.9 (Y4), U37.18 (DQ4), U39.18 (DQ4)
- net AD5: now also U31.7 (D5), U34.7 (Y5), U37.19 (DQ5), U39.19 (DQ5)
- net AD6: now also U31.8 (D6), U34.5 (Y6), U37.20 (DQ6), U39.20 (DQ6)
- net AD7: now also U31.9 (D7), U34.3 (Y7), U37.21 (DQ7), U39.21 (DQ7)
- net MEM_OE: now also U36.24 (OE), U37.24 (OE), U38.24 (OE), U39.24 (OE)
- net MEM_WE_H: now also U37.29 (WE), U39.29 (WE)
- net MEM_WE_L: now also U36.29 (WE), U38.29 (WE)
- net MST_WR: now also U30.12 (Q0), U34.2 (A0)
- net S100_A0: now also U29.3 (A0)
- net S100_A1: now also U29.4 (A1)
- net S100_A2: now also U29.10 (A2)
- net S100_A3: now also U28.2 (P0)
- net S100_A4: now also U28.4 (P1)
- net S100_A5: now also U28.6 (P2)
- net S100_A6: now also U28.8 (P3)
- net S100_ADSB: now also U5.65 (S100_ADSB); no longer U4.36 (S100_ADSB)
- net S100_A_OE: now also U5.69 (S100_A_OE); no longer U4.67 (S100_A_OE)
- net S100_CDSB: now also U5.68 (S100_CDSB); no longer U4.39 (S100_CDSB)
- net S100_C_OE: now also U5.73 (S100_C_OE); no longer U4.69 (S100_C_OE)
- net S100_DO0: now also U30.2 (D0)
- net S100_DO1: now also U30.3 (D1)
- net S100_DO2: now also U30.4 (D2)
- net S100_DO3: now also U30.5 (D3)
- net S100_DO4: now also U30.6 (D4)
- net S100_DO5: now also U30.7 (D5)
- net S100_DO6: now also U30.8 (D6)
- net S100_DO7: now also U30.9 (D7)
- net S100_INT: now also U4.36 (S100_INT); no longer U5.63 (S100_INT)
- net S100_NMI: now also U4.37 (S100_NMI); no longer U5.64 (S100_NMI)
- net S100_SDSB: now also U5.67 (S100_SDSB); no longer U4.37 (S100_SDSB)
- net S100_S_OE: now also U5.70 (S100_S_OE); no longer U4.68 (S100_S_OE)
- net S100_sINP: now also U29.6 (sINP)
- net S100_sOUT: now also U29.5 (sOUT)
- net SLAVE_ONLY: no longer U4.64 (SLAVE_ONLY)
- net Z_AS: no longer U4.12 (Z_AS)
- net Z_CLK: now also U29.1 (Z_CLK)
- net Z_INT: now also U4.39 (Z_INT); no longer U5.56 (Z_INT)
- net Z_NMI: now also U4.67 (Z_NMI); no longer U5.57 (Z_NMI)
- net Z280_INT_C: now reaches U1.26 (INT-C)
- net Z280_INT_C: now also U29.15 (MS_FULL)
- net GREQ: now reaches U1.30 (CTIO0/GREQ)
- net GREQ: now also U4.75 (GREQ)
- net GACK: now reaches U1.32 (CTIN0/GACK)
- net GACK: now also U4.76 (GACK)
- net Z280_INT_B: now reaches U1.36 (INT-B/EOP-B)
- net Z280_INT_B: now also U29.14 (INT_B)
- removed net A20: U1.45 (A20), U17.6 (A4), U23.11 (Q4), U24.11 (Q4), U24.12 (P4), U4.9 (A20)
- net A8 renamed A1_EFF
- net A1_EFF: now also U4.68 (A1_EFF), U29.8 (INT_CLR), U33.13 (Y2), U36.5 (A7), U37.5 (A7), U38.5 (A7), U39.5 (A7), U40.3 (A11)
- removed net MEM_CE0: U4.10 (MEM_CE0), U6.22 (CE), U7.22 (CE)
- removed net MEM_CE1: U4.8 (MEM_CE1), U8.22 (CE), U9.22 (CE)
- net S100_SIXTN renamed MS_BYTE3
- net MS_BYTE3: now also U30.15 (Q3), U34.8 (A3)
- net SLV_WR renamed MS_BYTE1
- net MS_BYTE1: now also U30.13 (Q1), U34.4 (A1)
- net SPLIT renamed MS_BYTE2
- net MS_BYTE2: now also U30.14 (Q2), U34.6 (A2)
- new net DR_0: J12.2 (SEL), U28.3 (Q0)
- new net DR_1: J13.2 (SEL), U28.5 (Q1)
- new net DR_2: J14.2 (SEL), U28.7 (Q2)
- new net DR_3: J15.2 (SEL), U28.9 (Q3)
- new net IWANT: U4.77 (IWANT)
- new net MINE: U4.12 (MINE), U5.63 (MINE)
- new net MODE: U4.64 (MODE), U5.74 (MODE)
- new net MS_BYTE7: U30.19 (Q7), U34.17 (A7)
- new net MS_SET: U29.18 (MS_SET), U30.11 (CLK)
- new net REG_BLOCK: U32.19 (PEQQ), U33.6 (G1)
- new net SM_BYTE0: U31.12 (Q0)
- new net SM_BYTE1: U31.13 (Q1)
- new net SM_BYTE2: U31.14 (Q2)
- new net SM_BYTE3: U31.15 (Q3)
- new net SM_BYTE4: U31.16 (Q4)
- new net SM_BYTE5: U31.17 (Q5)
- new net SM_BYTE6: U31.18 (Q6)
- new net SM_BYTE7: U31.19 (Q7)
- new net SM_SET: U29.19 (SM_SET), U31.11 (CLK)
- new net W: U29.20 (W), U35.6 (A2), U4.8 (W)
